File: Hardware/Production/Qwiic_TMF8801-Panel.brd (EAGLE design)
At the start: 123.2 x 117.3 mm, 822 parts, among them J1 Qwiic, J11 Qwiic, J12 Qwiic, J15 Qwiic, J16 Qwiic, J19 Qwiic, J2 Qwiic, J20 Qwiic, J23 Qwiic, J24 Qwiic, J27 Qwiic, J28 Qwiic, J31 Qwiic, J32 Qwiic, J35 Qwiic, J36 Qwiic, J39 Qwiic, J40 Qwiic, J43 Qwiic, J44 Qwiic, J47 Qwiic, J48 Qwiic, J51 Qwiic, J52 Qwiic, J55 Qwiic, J56 Qwiic, J59 Qwiic, J60 Qwiic, J63 Qwiic, J64 Qwiic, J7 Qwiic, J8 Qwiic, U1 TMF8801, U10 TMF8801, U11 TMF8801, U12 TMF8801, U13 TMF8801, U14 TMF8801, U15 TMF8801, U16 TMF8801, U2 TMF8801, U3 TMF8801, U4 TMF8801, U5 TMF8801, U6 TMF8801, U7 TMF8801, U8 TMF8801, U9 TMF8801

Commit message: Fixed inverted SCL and SDA files; created panelized version.
Connections:
- net SCL: now also R2.1, U1.5; no longer R1.1, U1.6
- net SCL1: now also R7.1, U2.5; no longer R6.1, U2.6
- net SCL10: now also R52.1, U11.5; no longer R51.1, U11.6
- net SCL11: now also R57.1, U12.5; no longer R56.1, U12.6
- net SCL12: now also R62.1, U13.5; no longer R61.1, U13.6
- net SCL13: now also R67.1, U14.5; no longer R66.1, U14.6
- net SCL14: now also R72.1, U15.5; no longer R71.1, U15.6
- net SCL15: now also R77.1, U16.5; no longer R76.1, U16.6
- net SCL2: now also R12.1, U3.5; no longer R11.1, U3.6
- net SCL3: now also R17.1, U4.5; no longer R16.1, U4.6
- net SCL4: now also R22.1, U5.5; no longer R21.1, U5.6
- net SCL5: now also R27.1, U6.5; no longer R26.1, U6.6
- net SCL6: now also R32.1, U7.5; no longer R31.1, U7.6
- net SCL7: now also R37.1, U8.5; no longer R36.1, U8.6
- net SCL8: now also R42.1, U9.5; no longer R41.1, U9.6
- net SCL9: now also R47.1, U10.5; no longer R46.1, U10.6
- net SDA: now also R1.1, U1.6; no longer R2.1, U1.5
- net SDA1: now also R6.1, U2.6; no longer R7.1, U2.5
- net SDA10: now also R51.1, U11.6; no longer R52.1, U11.5
- net SDA11: now also R56.1, U12.6; no longer R57.1, U12.5
- net SDA12: now also R61.1, U13.6; no longer R62.1, U13.5
- net SDA13: now also R66.1, U14.6; no longer R67.1, U14.5
- net SDA14: now also R71.1, U15.6; no longer R72.1, U15.5
- net SDA15: now also R76.1, U16.6; no longer R77.1, U16.5
- net SDA2: now also R11.1, U3.6; no longer R12.1, U3.5
- net SDA3: now also R16.1, U4.6; no longer R17.1, U4.5
- net SDA4: now also R21.1, U5.6; no longer R22.1, U5.5
- net SDA5: now also R26.1, U6.6; no longer R27.1, U6.5
- net SDA6: now also R31.1, U7.6; no longer R32.1, U7.5
- net SDA7: now also R36.1, U8.6; no longer R37.1, U8.5
- net SDA8: now also R41.1, U9.6; no longer R42.1, U9.5
- net SDA9: now also R46.1, U10.6; no longer R47.1, U10.5
Routing:
- net SCL15: track 56.8 -> 69.1 mm
- net SCL14: track 56.8 -> 69.1 mm
- net SCL13: track 56.8 -> 69.1 mm
- net SCL12: track 56.8 -> 69.1 mm
- net SCL9: track 56.8 -> 69.1 mm
- net SCL11: track 56.8 -> 69.1 mm
- net SCL6: track 56.8 -> 69.1 mm
- net SCL3: track 56.8 -> 69.1 mm
- net SCL2: track 56.8 -> 69.1 mm
- net SCL10: track 56.8 -> 69.1 mm
- net SCL8: track 56.8 -> 69.1 mm
- net SCL4: track 56.8 -> 69.1 mm
- net SCL7: track 56.8 -> 69.1 mm
- net SCL1: track 56.8 -> 69.1 mm
- net SCL: track 56.8 -> 69.1 mm
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Other:
- board text added: "x02"
- board text removed: "x01"
